File: GateWay_ver_2_1/PCB/Gateway_STM32_ver_2_0/Ethernet.kicad_sch (KiCad schematic)
At the start: 41 parts, among them J2 HR911105A, U16 TPD2EUSB30, U4 W5500, U5 TPD2EUSB30, Y3 25mhz

Commit message: 1
Parts:
- added C28: 0.1uF, Capacitor_SMD:C_0603_1608Metric, symbol Device:C
Connections:
- net GND: now also C28.1
- net W5500_RST: now also C28.2
Other:
- moved on the sheet: R17, R20
Changed lines of the file:
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@@
     )
   )
-  (global_label "W5500_INT" (shape input) (at 28.702 109.728 0) (fields_autoplaced)
+  (global_label "W5500_INT" (shape input) (at 20.955 108.331 0) (fields_autoplaced)
     (effects (font (size 1.27 1.27)) (justify left))
-    (property "Intersheet References" "${INTERSHEET_REFS}" (id 0) (at 41.1862 109.8074 0)
+    (property "Intersheet References" "${INTERSHEET_REFS}" (id 0) (at 33.4392 108.4104 0)
       (effects (font (size 1.27 1.27)) (justify left) hide)
     )
@@
     )
   )
-  (global_label "W5500_RST" (shape input) (at 33.655 104.521 0) (fields_autoplaced)
+  (global_label "W5500_RST" (shape input) (at 25.908 103.124 0) (fields_autoplaced)
     (effects (font (size 1.27 1.27)) (justify left))
-    (property "Intersheet References" "${INTERSHEET_REFS}" (id 0) (at 46.6835 104.6004 0)
+    (property "Intersheet References" "${INTERSHEET_REFS}" (id 0) (at 38.9365 103.2034 0)
       (effects (font (size 1.27 1.27)) (justify left) hide)
     )
@@
     )
   )
+  (global_label "W5500_RST" (shape input) (at 32.893 97.79 0) (fields_autoplaced)
+    (effects (font (size 1.27 1.27)) (justify left))
+    (property "Intersheet References" "${INTERSHEET_REFS}" (id 0) (at 45.9215 97.8694 0)
+      (effects (font (size 1.27 1.27)) (justify left) hide)
+    )
+  )
   (global_label "TRD1_P" (shape input) (at 255.27 151.384 180) (fields_autoplaced)
     (effects (font (size 1.27 1.27)) (justify right))
@@
     (pin "2")
   )
-  (symbol (lib_id "Device:R") (at 28.702 105.918 180) (unit 1)
-    (in_bom yes) (on_board yes)
-    (property "Reference" "R20" (id 0) (at 30.607 105.029 90)
-      (effects (font (size 1.27 1.27)) (justify left))
-    )
-    (property "Value" "1k" (id 1) (at 28.702 104.775 90)
-      (effects (font (size 1.27 1.27)) (justify left))
-    )
-    (property "Footprint" "Resistor_SMD:R_0603_1608Metric" (id 2) (at 30.48 105.918 90)
-      (effects (font (size 1.27 1.27)) hide)
-    )
-    (property "Datasheet" "~" (id 3) (at 28.702 105.918 0)
+  (symbol (lib_id "Device:R") (at 20.955 104.521 180) (unit 1)
+    (in_bom yes) (on_board yes)
+    (property "Reference" "R20" (id 0) (at 22.86 103.632 90)
+      (effects (font (size 1.27 1.27)) (justify left))
+    )
+    (property "Value" "1k" (id 1) (at 20.955 103.378 90)
+      (effects (font (size 1.27 1.27)) (justify left))
+    )
+    (property "Footprint" "Resistor_SMD:R_0603_1608Metric" (id 2) (at 22.733 104.521 90)
+      (effects (font (size 1.27 1.27)) hide)
+    )
+    (property "Datasheet" "~" (id 3) (at 20.955 104.521 0)
       (effects (font (size 1.27 1.27)) hide)
     )
@@
     (pin "1")
   )
-  (symbol (lib_id "power:+3.3V") (at 28.702 102.108 0) (unit 1)
-    (in_bom yes) (on_board yes)
-    (property "Reference" "#PWR0223" (id 0) (at 28.702 105.918 0)
-      (effects (font (size 1.27 1.27)) hide)
-    )
-    (property "Value" "+3.3V" (id 1) (at 28.702 96.52 90))
-    (property "Footprint" "" (id 2) (at 28.702 102.108 0)
-      (effects (font (size 1.27 1.27)) hide)
-    )
-    (property "Datasheet" "" (id 3) (at 28.702 102.108 0)
+  (symbol (lib_id "Device:C") (at 32.893 93.98 0) (unit 1)
+    (in_bom yes) (on_board yes)
+    (property "Reference" "C28" (id 0) (at 35.814 92.8116 0)
+      (effects (font (size 1.27 1.27)) (justify left))
+    )
+    (property "Value" "0.1uF" (id 1) (at 29.591 96.647 90)
+      (effects (font (size 1.27 1.27)) (justify left))
+    )
+    (property "Footprint" "Capacitor_SMD:C_0603_1608Metric" (id 2) (at 33.8582 97.79 0)
+      (effects (font (size 1.27 1.27)) hide)
+    )
+    (property "Datasheet" "~" (id 3) (at 32.893 93.98 0)
+      (effects (font (size 1.27 1.27)) hide)
+    )
+    (pin "1")
+    (pin "2")
+  )
+  (symbol (lib_id "power:+3.3V") (at 20.955 100.711 0) (unit 1)
+    (in_bom yes) (on_board yes)
+    (property "Reference" "#PWR0223" (id 0) (at 20.955 104.521 0)
+      (effects (font (size 1.27 1.27)) hide)
+    )
+    (property "Value" "+3.3V" (id 1) (at 20.955 95.123 90))
+    (property "Footprint" "" (id 2) (at 20.955 100.711 0)
+      (effects (font (size 1.27 1.27)) hide)
+    )
+    (property "Datasheet" "" (id 3) (at 20.955 100.711 0)
       (effects (font (size 1.27 1.27)) hide)
     )
@@
     (pin "1")
   )
+  (symbol (lib_id "power:GND") (at 32.893 90.17 180) (unit 1)
+    (in_bom yes) (on_board yes)
+    (property "Reference" "#PWR0292" (id 0) (at 32.893 83.82 0)
+      (effects (font (size 1.27 1.27)) hide)
+    )
+    (property "Value" "GND" (id 1) (at 32.893 85.471 90))
+    (property "Footprint" "" (id 2) (at 32.893 90.17 0)
+      (effects (font (size 1.27 1.27)) hide)
+    )
+    (property "Datasheet" "" (id 3) (at 32.893 90.17 0)
+      (effects (font (size 1.27 1.27)) hide)
+    )
+    (pin "1")
+  )
   (symbol (lib_id "power:+3.3VP") (at 62.865 65.913 0) (unit 1)
     (in_bom yes) (on_board yes)
@@
     (pin "1")
   )
-  (symbol (lib_id "Device:R") (at 33.655 100.711 180) (unit 1)
-    (in_bom yes) (on_board yes)
-    (property "Reference" "R17" (id 0) (at 35.56 99.822 90)
-      (effects (font (size 1.27 1.27)) (justify left))
-    )
-    (property "Value" "1k" (id 1) (at 33.655 99.568 90)
-      (effects (font (size 1.27 1.27)) (justify left))
-    )
-    (property "Footprint" "Resistor_SMD:R_0603_1608Metric" (id 2) (at 35.433 100.711 90)
-      (effects (font (size 1.27 1.27)) hide)
-    )
-    (property "Datasheet" "~" (id 3) (at 33.655 100.711 0)
+  (symbol (lib_id "Device:R") (at 25.908 99.314 180) (unit 1)
+    (in_bom yes) (on_board yes)
+    (property "Reference" "R17" (id 0) (at 27.813 98.425 90)
+      (effects (font (size 1.27 1.27)) (justify left))
+    )
+    (property "Value" "1k" (id 1) (at 25.908 98.171 90)
+      (effects (font (size 1.27 1.27)) (justify left))
+    )
+    (property "Footprint" "Resistor_SMD:R_0603_1608Metric" (id 2) (at 27.686 99.314 90)
+      (effects (font (size 1.27 1.27)) hide)
+    )
+    (property "Datasheet" "~" (id 3) (at 25.908 99.314 0)
       (effects (font (size 1.27 1.27)) hide)
     )
@@
     (pin "1")
   )
-  (symbol (lib_id "power:+3.3V") (at 33.655 96.901 0) (unit 1)
-    (in_bom yes) (on_board yes)
-    (property "Reference" "#PWR0224" (id 0) (at 33.655 100.711 0)
-      (effects (font (size 1.27 1.27)) hide)
-    )
-    (property "Value" "+3.3V" (id 1) (at 33.655 91.313 90))
-    (property "Footprint" "" (id 2) (at 33.655 96.901 0)
-      (effects (font (size 1.27 1.27)) hide)
-    )
-    (property "Datasheet" "" (id 3) (at 33.655 96.901 0)
-      (effects (font (size 1.27 1.27)) hide)
-    )
+  (symbol (lib_id "power:+3.3V") (at 25.908 95.504 0) (unit 1)
+    (in_bom yes) (on_board yes)
+    (property "Reference" "#PWR0224" (id 0) (at 25.908 99.314 0)
+      (effects (font (size 1.27 1.27)) hide)
+    )
+    (property "Value" "+3.3V" (id 1) (at 25.908 89.916 90))
+    (property "Footprint" "" (id 2) (at 25.908 95.504 0)
+      (effects (font (size 1.27 1.27)) hide)
+    )
+    (property "Datasheet" "" (id 3) (at 25.908 95.504 0)
+      (effects (font (size 1.27 1.27)) hide)
+    )
