File: GateWay_ver_2_1/PCB/Gateway_STM32_ver_2_0/Ext Connectors.kicad_sch (KiCad schematic)
At the start: 2 parts, among them J10 Conn_02x10_Odd_Even, J11 Conn_01x05

Commit message: 1
Parts:
- added R106, R107: 10k, Resistor_SMD:R_0603_1608Metric, symbol Device:R
Connections:
- net +3V3: now also R106.2, R107.2
- net Nextion_Rx: now also R106.1
- net Nextion_Tx: now also R107.1
Changed lines of the file:
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@@
+    )
+  )
+  (global_label "Nextion_Tx" (shape input) (at 126.746 77.216 180) (fields_autoplaced)
+    (effects (font (size 1.27 1.27)) (justify right))
+    (property "Intersheet References" "${INTERSHEET_REFS}" (id 0) (at 114.3828 77.1366 0)
+      (effects (font (size 1.27 1.27)) (justify right) hide)
+    )
+  )
+  (global_label "Nextion_Rx" (shape input) (at 126.746 70.485 180) (fields_autoplaced)
+    (effects (font (size 1.27 1.27)) (justify right))
+    (property "Intersheet References" "${INTERSHEET_REFS}" (id 0) (at 114.0804 70.4056 0)
+      (effects (font (size 1.27 1.27)) (justify right) hide)
     )
   )
@@
     (pin "1")
   )
+  (symbol (lib_id "power:+3.3V") (at 134.366 70.485 270) (mirror x) (unit 1)
+    (in_bom yes) (on_board yes)
+    (property "Reference" "#PWR0310" (id 0) (at 130.556 70.485 0)
+      (effects (font (size 1.27 1.27)) hide)
+    )
+    (property "Value" "+3.3V" (id 1) (at 139.7 70.485 90))
+    (property "Footprint" "" (id 2) (at 134.366 70.485 0)
+      (effects (font (size 1.27 1.27)) hide)
+    )
+    (property "Datasheet" "" (id 3) (at 134.366 70.485 0)
+      (effects (font (size 1.27 1.27)) hide)
+    )
+    (pin "1")
+  )
   (symbol (lib_id "power:GND") (at 75.438 83.947 90) (unit 1)
     (in_bom yes) (on_board yes)
@@
     )
     (pin "1")
+  )
+  (symbol (lib_id "power:+3.3V") (at 134.366 77.216 270) (mirror x) (unit 1)
+    (in_bom yes) (on_board yes)
+    (property "Reference" "#PWR0311" (id 0) (at 130.556 77.216 0)
+      (effects (font (size 1.27 1.27)) hide)
+    )
+    (property "Value" "+3.3V" (id 1) (at 139.827 77.216 90))
+    (property "Footprint" "" (id 2) (at 134.366 77.216 0)
+      (effects (font (size 1.27 1.27)) hide)
+    )
+    (property "Datasheet" "" (id 3) (at 134.366 77.216 0)
+      (effects (font (size 1.27 1.27)) hide)
+    )
+    (pin "1")
+  )
+  (symbol (lib_id "Device:R") (at 130.556 77.216 90) (mirror x) (unit 1)
+    (in_bom yes) (on_board yes)
+    (property "Reference" "R107" (id 0) (at 133.096 75.057 90)
+      (effects (font (size 1.27 1.27)) (justify left))
+    )
+    (property "Value" "10k" (id 1) (at 132.08 77.216 90)
+      (effects (font (size 1.27 1.27)) (justify left))
+    )
+    (property "Footprint" "Resistor_SMD:R_0603_1608Metric" (id 2) (at 130.556 75.438 90)
+      (effects (font (size 1.27 1.27)) hide)
+    )
+    (property "Datasheet" "~" (id 3) (at 130.556 77.216 0)
+      (effects (font (size 1.27 1.27)) hide)
+    )
+    (pin "1")
+    (pin "2")
   )
   (symbol (lib_id "power:GND") (at 137.414 98.679 270) (unit 1)
@@
     (pin "1")
   )
+  (symbol (lib_id "Device:R") (at 130.556 70.485 90) (mirror x) (unit 1)
+    (in_bom yes) (on_board yes)
+    (property "Reference" "R106" (id 0) (at 133.096 68.326 90)
+      (effects (font (size 1.27 1.27)) (justify left))
+    )
+    (property "Value" "10k" (id 1) (at 132.334 70.485 90)
+      (effects (font (size 1.27 1.27)) (justify left))
+    )
+    (property "Footprint" "Resistor_SMD:R_0603_1608Metric" (id 2) (at 130.556 68.707 90)
+      (effects (font (size 1.27 1.27)) hide)
+    )
+    (property "Datasheet" "~" (id 3) (at 130.556 70.485 0)
+      (effects (font (size 1.27 1.27)) hide)
+    )
+    (pin "1")
+    (pin "2")
+  )
   (symbol (lib_id "Connector_Generic:Conn_02x10_Odd_Even") (at 67.818 89.027 0) (unit 1)
