File: GateWay_ver_2_1/PCB/Gateway_STM32_ver_2_0/RS-485 & 232.kicad_sch (KiCad schematic)
At the start: 37 parts, among them J12 RJ45_LED_Shielded, J6 RJ45_LED_Shielded, J7 RJ45_LED_Shielded, Q5 MMBT3906, Q6 MMBT3906, Q7 MMBT3906, Q8 MMBT3906, SW3 SW_Push, U10 MAX3485, U11 SN74LV4052APW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

Commit message: 1
Connections:
- net 485_N: now also D23.1 (A1); no longer D23.2 (A2)
- net 485_P: now also D23.2 (A2); no longer D23.1 (A1)
Changed lines of the file:
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@@
     )
   )
-  (global_label "485_P" (shape input) (at 225.552 161.29 0) (fields_autoplaced)
-    (effects (font (size 1.27 1.27)) (justify left))
-    (property "Intersheet References" "${INTERSHEET_REFS}" (id 0) (at 136.652 -218.44 0)
+  (global_label "485_P" (shape input) (at 207.772 161.29 180) (fields_autoplaced)
+    (effects (font (size 1.27 1.27)) (justify right))
+    (property "Intersheet References" "${INTERSHEET_REFS}" (id 0) (at 296.672 541.02 0)
       (effects (font (size 1.27 1.27)) hide)
     )
@@
     )
   )
-  (global_label "485_N" (shape input) (at 207.772 161.29 180) (fields_autoplaced)
-    (effects (font (size 1.27 1.27)) (justify right))
-    (property "Intersheet References" "${INTERSHEET_REFS}" (id 0) (at 296.672 558.8 0)
+  (global_label "485_N" (shape input) (at 225.552 161.29 0) (fields_autoplaced)
+    (effects (font (size 1.27 1.27)) (justify left))
+    (property "Intersheet References" "${INTERSHEET_REFS}" (id 0) (at 136.652 -236.22 0)
       (effects (font (size 1.27 1.27)) hide)
     )

Commit message: 1
Parts:
- added R108, R109: 10k, Resistor_SMD:R_0603_1608Metric, symbol Device:R
Connections:
- net +3V3: now also R108.2, R109.2
- net 485_N: now also R108.1
- net 485_P: now also R109.1
Changed lines of the file:
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@@
     (effects (font (size 5.0038 5.0038) (thickness 1.0008) bold) (justify left bottom))
   )
+  (global_label "485_P" (shape input) (at 237.8202 134.874 270) (fields_autoplaced)
+    (effects (font (size 1.27 1.27)) (justify right))
+    (property "Intersheet References" "${INTERSHEET_REFS}" (id 0) (at 592.1502 214.249 90)
+      (effects (font (size 1.27 1.27)) (justify right) hide)
+    )
+  )
   (global_label "485_N" (shape input) (at 174.117 188.341 270) (fields_autoplaced)
     (effects (font (size 1.27 1.27)) (justify right))
@@
     (effects (font (size 1.27 1.27)) (justify right))
     (property "Intersheet References" "${INTERSHEET_REFS}" (id 0) (at 18.1954 122.8566 0)
+      (effects (font (size 1.27 1.27)) (justify right) hide)
+    )
+  )
+  (global_label "485_N" (shape input) (at 231.0892 134.874 270) (fields_autoplaced)
+    (effects (font (size 1.27 1.27)) (justify right))
+    (property "Intersheet References" "${INTERSHEET_REFS}" (id 0) (at 575.8942 214.249 90)
       (effects (font (size 1.27 1.27)) (justify right) hide)
     )
@@
     (pin "3")
   )
+  (symbol (lib_id "power:+3.3V") (at 237.8202 127.254 0) (mirror y) (unit 1)
+    (in_bom yes) (on_board yes)
+    (property "Reference" "#PWR0313" (id 0) (at 237.8202 131.064 0)
+      (effects (font (size 1.27 1.27)) hide)
+    )
+    (property "Value" "+3.3V" (id 1) (at 237.8202 123.444 0))
+    (property "Footprint" "" (id 2) (at 237.8202 127.254 0)
+      (effects (font (size 1.27 1.27)) hide)
+    )
+    (property "Datasheet" "" (id 3) (at 237.8202 127.254 0)
+      (effects (font (size 1.27 1.27)) hide)
+    )
+    (pin "1")
+  )
+  (symbol (lib_id "Device:R") (at 237.8202 131.064 0) (mirror x) (unit 1)
+    (in_bom yes) (on_board yes)
+    (property "Reference" "R109" (id 0) (at 235.6612 128.524 90)
+      (effects (font (size 1.27 1.27)) (justify left))
+    )
+    (property "Value" "10k" (id 1) (at 237.8202 129.54 90)
+      (effects (font (size 1.27 1.27)) (justify left))
+    )
+    (property "Footprint" "Resistor_SMD:R_0603_1608Metric" (id 2) (at 236.0422 131.064 90)
+      (effects (font (size 1.27 1.27)) hide)
+    )
+    (property "Datasheet" "~" (id 3) (at 237.8202 131.064 0)
+      (effects (font (size 1.27 1.27)) hide)
+    )
+    (pin "1")
+    (pin "2")
+  )
   (symbol (lib_id "Transistor_BJT:MMBT3906") (at 117.094 64.516 0) (mirror x) (unit 1)
     (in_bom yes) (on_board yes) (fields_autoplaced)
@@
     (pin "1")
   )
+  (symbol (lib_id "power:+3.3V") (at 231.0892 127.254 0) (mirror y) (unit 1)
+    (in_bom yes) (on_board yes)
+    (property "Reference" "#PWR0312" (id 0) (at 231.0892 131.064 0)
+      (effects (font (size 1.27 1.27)) hide)
+    )
+    (property "Value" "+3.3V" (id 1) (at 231.0892 123.444 0))
+    (property "Footprint" "" (id 2) (at 231.0892 127.254 0)
+      (effects (font (size 1.27 1.27)) hide)
+    )
+    (property "Datasheet" "" (id 3) (at 231.0892 127.254 0)
+      (effects (font (size 1.27 1.27)) hide)
+    )
+    (pin "1")
+  )
   (symbol (lib_id "Device:R") (at 38.481 127.508 180) (unit 1)
     (in_bom yes) (on_board yes)
@@
       (effects (font (size 1.27 1.27)) hide)
     )
+    (pin "1")
+    (pin "2")
+  )
+  (symbol (lib_id "Device:R") (at 231.0892 131.064 0) (mirror x) (unit 1)
+    (in_bom yes) (on_board yes)
+    (property "Reference" "R108" (id 0) (at 228.9302 128.524 90)
+      (effects (font (size 1.27 1.27)) (justify left))
+    )
+    (property "Value" "10k" (id 1) (at 231.0892 129.286 90)
+      (effects (font (size 1.27 1.27)) (justify left))
+    )
+    (property "Footprint" "Resistor_SMD:R_0603_1608Metric" (id 2) (at 229.3112 131.064 90)
+      (effects (font (size 1.27 1.27)) hide)
+    )
+    (property "Datasheet" "~" (id 3) (at 231.0892 131.064 0)
+      (effects (font (size 1.27 1.27)) hide)
+    )
