File: GateWay_ver_2_1/PCB/Gateway_STM32_ver_2_0/EEPROM.kicad_sch (KiCad schematic)
At the start: 4 parts, among them U13 CAT24C256

Commit message: 1
Connections:
- net SCL is gone; now on net I2C2_SCL: R71.2
- net SDA is gone; now on net I2C2_SDA: R72.2
Changed lines of the file:
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@@
     (effects (font (size 5.0038 5.0038) (thickness 1.0008) bold) (justify left bottom))
   )
-  (global_label "SCL" (shape input) (at 58.674 38.862 270) (fields_autoplaced)
+  (global_label "I2C2_SDA" (shape input) (at 66.294 38.862 270) (fields_autoplaced)
     (effects (font (size 1.27 1.27)) (justify right))
-    (property "Intersheet References" "${INTERSHEET_REFS}" (id 0) (at -497.586 -514.858 0)
-      (effects (font (size 1.27 1.27)) hide)
+    (property "Intersheet References" "${INTERSHEET_REFS}" (id 0) (at 66.2146 50.0157 90)
+      (effects (font (size 1.27 1.27)) (justify right) hide)
     )
   )
@@
     )
   )
-  (global_label "SDA" (shape input) (at 66.294 38.862 270) (fields_autoplaced)
+  (global_label "I2C2_SCL" (shape input) (at 58.674 38.862 270) (fields_autoplaced)
     (effects (font (size 1.27 1.27)) (justify right))
-    (property "Intersheet References" "${INTERSHEET_REFS}" (id 0) (at -497.586 -514.858 0)
-      (effects (font (size 1.27 1.27)) hide)
+    (property "Intersheet References" "${INTERSHEET_REFS}" (id 0) (at 58.5946 49.9552 90)
+      (effects (font (size 1.27 1.27)) (justify right) hide)
     )
   )

Commit message: 1
Parts:
- added C115: 0.1uF, Capacitor_SMD:C_0603_1608Metric, symbol Device:C
- added U26: 24AA02E48, Package_TO_SOT_SMD:SOT-23-6, symbol Symbols:24AA02E48
Connections:
- net +3V3: now also C115.1, U26.6 (VCC)
- net GND: now also C115.2, U26.2 (GND), U26.4 (A1), U26.5 (A0)
- net I2C2_SCL: now also U26.1 (SCL)
- net I2C2_SDA: now also U26.3 (SDA)
Changed lines of the file:
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@@
     (effects (font (size 5.0038 5.0038) (thickness 1.0008) bold) (justify left bottom))
+  )
+  (global_label "I2C2_SDA" (shape input) (at 129.667 46.609 0) (fields_autoplaced)
+    (effects (font (size 1.27 1.27)) (justify left))
+    (property "Intersheet References" "${INTERSHEET_REFS}" (id 0) (at 140.8207 46.6884 0)
+      (effects (font (size 1.27 1.27)) (justify left) hide)
+    )
   )
   (global_label "I2C2_SDA" (shape input) (at 66.294 38.862 270) (fields_autoplaced)
@@
     )
   )
+  (global_label "I2C2_SCL" (shape input) (at 129.667 38.989 0) (fields_autoplaced)
+    (effects (font (size 1.27 1.27)) (justify left))
+    (property "Intersheet References" "${INTERSHEET_REFS}" (id 0) (at 140.7602 39.0684 0)
+      (effects (font (size 1.27 1.27)) (justify left) hide)
+    )
+  )
+  (symbol (lib_id "power:GND") (at 114.427 42.799 270) (unit 1)
+    (in_bom yes) (on_board yes)
+    (property "Reference" "#PWR0315" (id 0) (at 108.077 42.799 0)
+      (effects (font (size 1.27 1.27)) hide)
+    )
+    (property "Value" "GND" (id 1) (at 110.0328 42.926 90))
+    (property "Footprint" "" (id 2) (at 114.427 42.799 0)
+      (effects (font (size 1.27 1.27)) hide)
+    )
+    (property "Datasheet" "" (id 3) (at 114.427 42.799 0)
+      (effects (font (size 1.27 1.27)) hide)
+    )
+    (pin "1")
+  )
   (symbol (lib_id "power:+3.3V") (at 58.674 31.242 0) (unit 1)
     (in_bom yes) (on_board yes)
@@
     (pin "1")
   )
+  (symbol (lib_id "power:+3.3V") (at 126.111 25.527 270) (unit 1)
+    (in_bom yes) (on_board yes)
+    (property "Reference" "#PWR0313" (id 0) (at 122.301 25.527 0)
+      (effects (font (size 1.27 1.27)) hide)
+    )
+    (property "Value" "+3.3V" (id 1) (at 131.572 25.527 90))
+    (property "Footprint" "" (id 2) (at 126.111 25.527 0)
+      (effects (font (size 1.27 1.27)) hide)
+    )
+    (property "Datasheet" "" (id 3) (at 126.111 25.527 0)
+      (effects (font (size 1.27 1.27)) hide)
+    )
+    (pin "1")
+  )
   (symbol (lib_id "power:GND") (at 21.717 21.59 270) (unit 1)
     (in_bom yes) (on_board yes)
@@
     (pin "1")
   )
+  (symbol (lib_id "Symbols:24AA02E48") (at 122.047 42.799 0) (unit 1)
+    (in_bom yes) (on_board yes) (fields_autoplaced)
+    (property "Reference" "U26" (id 0) (at 122.047 32.6095 0))
+    (property "Value" "24AA02E48" (id 1) (at 122.047 35.3846 0))
+    (property "Footprint" "Package_TO_SOT_SMD:SOT-23-6" (id 2) (at 122.047 32.639 0)
+      (effects (font (size 1.27 1.27)) hide)
+    )
+    (property "Datasheet" "" (id 3) (at 122.047 32.639 0)
+      (effects (font (size 1.27 1.27)) hide)
+    )
+    (pin "1")
+    (pin "2")
+    (pin "3")
+    (pin "4")
+    (pin "5")
+    (pin "6")
+  )
   (symbol (lib_id "power:+3.3V") (at 33.782 31.115 0) (unit 1)
     (in_bom yes) (on_board yes)
@@
     (pin "2")
   )
+  (symbol (lib_id "power:GND") (at 122.047 52.959 0) (unit 1)
+    (in_bom yes) (on_board yes)
+    (property "Reference" "#PWR0317" (id 0) (at 122.047 59.309 0)
+      (effects (font (size 1.27 1.27)) hide)
+    )
+    (property "Value" "GND" (id 1) (at 122.174 57.3532 90))
+    (property "Footprint" "" (id 2) (at 122.047 52.959 0)
+      (effects (font (size 1.27 1.27)) hide)
+    )
+    (property "Datasheet" "" (id 3) (at 122.047 52.959 0)
+      (effects (font (size 1.27 1.27)) hide)
+    )
+    (pin "1")
+  )
   (symbol (lib_id "power:GND") (at 23.622 41.275 270) (unit 1)
     (in_bom yes) (on_board yes)
@@
     )
     (property "Datasheet" "" (id 3) (at 23.622 36.195 0)
+      (effects (font (size 1.27 1.27)) hide)
+    )
+    (pin "1")
+  )
+  (symbol (lib_id "power:+3.3V") (at 114.427 46.609 90) (unit 1)
+    (in_bom yes) (on_board yes)
+    (property "Reference" "#PWR0316" (id 0) (at 118.237 46.609 0)
+      (effects (font (size 1.27 1.27)) hide)
+    )
+    (property "Value" "+3.3V" (id 1) (at 108.839 46.609 90))
+    (property "Footprint" "" (id 2) (at 114.427 46.609 0)
+      (effects (font (size 1.27 1.27)) hide)
+    )
+    (property "Datasheet" "" (id 3) (at 114.427 46.609 0)
       (effects (font (size 1.27 1.27)) hide)
     )
@@
     (pin "1")
   )
+  (symbol (lib_id "power:GND") (at 114.427 38.989 270) (unit 1)
+    (in_bom yes) (on_board yes)
+    (property "Reference" "#PWR0314" (id 0) (at 108.077 38.989 0)
+      (effects (font (size 1.27 1.27)) hide)
+    )
+    (property "Value" "GND" (id 1) (at 110.0328 39.116 90))
+    (property "Footprint" "" (id 2) (at 114.427 38.989 0)
+      (effects (font (size 1.27 1.27)) hide)
+    )
+    (property "Datasheet" "" (id 3) (at 114.427 38.989 0)
+      (effects (font (size 1.27 1.27)) hide)
+    )
+    (pin "1")
+  )
+  (symbol (lib_id "power:GND") (at 118.491 25.527 270) (unit 1)
+    (in_bom yes) (on_board yes)
+    (property "Reference" "#PWR0312" (id 0) (at 112.141 25.527 0)
+      (effects (font (size 1.27 1.27)) hide)
+    )
+    (property "Value" "GND" (id 1) (at 114.0968 25.654 90))
+    (property "Footprint" "" (id 2) (at 118.491 25.527 0)
+      (effects (font (size 1.27 1.27)) hide)
+    )
+    (property "Datasheet" "" (id 3) (at 118.491 25.527 0)
+      (effects (font (size 1.27 1.27)) hide)
+    )
+    (pin "1")
+  )
+  (symbol (lib_id "Device:C") (at 122.301 25.527 270) (unit 1)
+    (in_bom yes) (on_board yes)
+    (property "Reference" "C115" (id 0) (at 123.4694 28.448 90)
+      (effects (font (size 1.27 1.27)) (justify left))
+    )
+    (property "Value" "0.1uF" (id 1) (at 117.221 28.702 90)
+      (effects (font (size 1.27 1.27)) (justify left))
+    )
+    (property "Footprint" "Capacitor_SMD:C_0603_1608Metric" (id 2) (at 118.491 26.4922 0)
+      (effects (font (size 1.27 1.27)) hide)
+    )
+    (property "Datasheet" "~" (id 3) (at 122.301 25.527 0)
+      (effects (font (size 1.27 1.27)) hide)
+    )
+    (pin "1")
+    (pin "2")
+  )
   (symbol (lib_id "Device:R") (at 66.294 35.052 0) (unit 1)

Commit message: 1
Parts:
- removed U26: 24AA02E48, Package_TO_SOT_SMD:SOT-23-6, symbol Symbols:24AA02E48
- added R? (x2): 4.7k, Resistor_SMD:R_0603_1608Metric, symbol Device:R
- added U?: 24AA02E48, Package_TO_SOT_SMD:SOT-23-5, symbol Symbols:24AA02E48
Connections:
- net +3V3: now also R?.1, R?.1, U?.4 (VCC)
- net GND: now also U?.2 (GND)
- new net I2C1_SCL: R?.2, U?.1 (SCL)
- new net I2C1_SDA: R?.2, U?.3 (SDA)
Changed lines of the file:
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@@
     (effects (font (size 5.0038 5.0038) (thickness 1.0008) bold) (justify left bottom))
-  )
-  (global_label "I2C2_SDA" (shape input) (at 129.667 46.609 0) (fields_autoplaced)
-    (effects (font (size 1.27 1.27)) (justify left))
-    (property "Intersheet References" "${INTERSHEET_REFS}" (id 0) (at 140.8207 46.6884 0)
-      (effects (font (size 1.27 1.27)) (justify left) hide)
-    )
   )
   (global_label "I2C2_SDA" (shape input) (at 66.294 38.862 270) (fields_autoplaced)
@@
     )
   )
+  (global_label "I2C1_SCL" (shape input) (at 152.4 34.29 270) (fields_autoplaced)
+    (effects (font (size 1.27 1.27)) (justify right))
+    (property "Intersheet References" "${INTERSHEET_REFS}" (id 0) (at 152.3206 45.3832 90)
+      (effects (font (size 1.27 1.27)) (justify right) hide)
+    )
+  )
   (global_label "I2C2_SCL" (shape input) (at 43.942 38.735 0) (fields_autoplaced)
     (effects (font (size 1.27 1.27)) (justify left))
@@
     )
   )
+  (global_label "I2C1_SDA" (shape input) (at 160.02 34.29 270) (fields_autoplaced)
+    (effects (font (size 1.27 1.27)) (justify right))
+    (property "Intersheet References" "${INTERSHEET_REFS}" (id 0) (at 159.9406 45.4437 90)
+      (effects (font (size 1.27 1.27)) (justify right) hide)
+    )
+  )
   (global_label "WP" (shape input) (at 43.942 41.275 0) (fields_autoplaced)
     (effects (font (size 1.27 1.27)) (justify left))
     (property "Intersheet References" "${INTERSHEET_REFS}" (id 0) (at -500.253 -514.985 0)
       (effects (font (size 1.27 1.27)) hide)
+    )
+  )
+  (global_label "I2C1_SCL" (shape input) (at 131.318 50.927 0) (fields_autoplaced)
+    (effects (font (size 1.27 1.27)) (justify left))
+    (property "Intersheet References" "${INTERSHEET_REFS}" (id 0) (at 142.4112 51.0064 0)
+      (effects (font (size 1.27 1.27)) (justify left) hide)
     )
   )
@@
     )
   )
+  (global_label "I2C1_SDA" (shape input) (at 131.318 44.577 0) (fields_autoplaced)
+    (effects (font (size 1.27 1.27)) (justify left))
+    (property "Intersheet References" "${INTERSHEET_REFS}" (id 0) (at 142.4717 44.6564 0)
+      (effects (font (size 1.27 1.27)) (justify left) hide)
+    )
+  )
   (global_label "I2C2_SDA" (shape input) (at 43.942 36.195 0) (fields_autoplaced)
     (effects (font (size 1.27 1.27)) (justify left))
@@
     )
   )
-  (global_label "I2C2_SCL" (shape input) (at 129.667 38.989 0) (fields_autoplaced)
-    (effects (font (size 1.27 1.27)) (justify left))
-    (property "Intersheet References" "${INTERSHEET_REFS}" (id 0) (at 140.7602 39.0684 0)
-      (effects (font (size 1.27 1.27)) (justify left) hide)
-    )
-  )
-  (symbol (lib_id "power:GND") (at 114.427 42.799 270) (unit 1)
-    (in_bom yes) (on_board yes)
-    (property "Reference" "#PWR0315" (id 0) (at 108.077 42.799 0)
-      (effects (font (size 1.27 1.27)) hide)
-    )
-    (property "Value" "GND" (id 1) (at 110.0328 42.926 90))
-    (property "Footprint" "" (id 2) (at 114.427 42.799 0)
-      (effects (font (size 1.27 1.27)) hide)
-    )
-    (property "Datasheet" "" (id 3) (at 114.427 42.799 0)
-      (effects (font (size 1.27 1.27)) hide)
-    )
-    (pin "1")
-  )
   (symbol (lib_id "power:+3.3V") (at 58.674 31.242 0) (unit 1)
     (in_bom yes) (on_board yes)
@@
     (pin "1")
   )
+  (symbol (lib_id "power:+3.3V") (at 116.078 43.307 90) (unit 1)
+    (in_bom yes) (on_board yes)
+    (property "Reference" "#PWR?" (id 0) (at 119.888 43.307 0)
+      (effects (font (size 1.27 1.27)) hide)
+    )
+    (property "Value" "+3.3V" (id 1) (at 110.617 43.307 90))
+    (property "Footprint" "" (id 2) (at 116.078 43.307 0)
+      (effects (font (size 1.27 1.27)) hide)
+    )
+    (property "Datasheet" "" (id 3) (at 116.078 43.307 0)
+      (effects (font (size 1.27 1.27)) hide)
+    )
+    (pin "1")
+  )
   (symbol (lib_id "Device:C") (at 25.527 21.59 270) (unit 1)
     (in_bom yes) (on_board yes)
@@
     (pin "1")
   )
-  (symbol (lib_id "Symbols:24AA02E48") (at 122.047 42.799 0) (unit 1)
-    (in_bom yes) (on_board yes) (fields_autoplaced)
-    (property "Reference" "U26" (id 0) (at 122.047 32.6095 0))
-    (property "Value" "24AA02E48" (id 1) (at 122.047 35.3846 0))
-    (property "Footprint" "Package_TO_SOT_SMD:SOT-23-6" (id 2) (at 122.047 32.639 0)
-      (effects (font (size 1.27 1.27)) hide)
-    )
-    (property "Datasheet" "" (id 3) (at 122.047 32.639 0)
-      (effects (font (size 1.27 1.27)) hide)
-    )
-    (pin "1")
-    (pin "2")
-    (pin "3")
-    (pin "4")
-    (pin "5")
-    (pin "6")
+  (symbol (lib_id "power:GND") (at 123.698 57.277 0) (unit 1)
+    (in_bom yes) (on_board yes)
+    (property "Reference" "#PWR?" (id 0) (at 123.698 63.627 0)
+      (effects (font (size 1.27 1.27)) hide)
+    )
+    (property "Value" "GND" (id 1) (at 123.825 61.6712 90))
+    (property "Footprint" "" (id 2) (at 123.698 57.277 0)
+      (effects (font (size 1.27 1.27)) hide)
+    )
+    (property "Datasheet" "" (id 3) (at 123.698 57.277 0)
+      (effects (font (size 1.27 1.27)) hide)
+    )
+    (pin "1")
   )
   (symbol (lib_id "power:+3.3V") (at 33.782 31.115 0) (unit 1)
@@
     (pin "2")
   )
-  (symbol (lib_id "power:GND") (at 122.047 52.959 0) (unit 1)
-    (in_bom yes) (on_board yes)
-    (property "Reference" "#PWR0317" (id 0) (at 122.047 59.309 0)
-      (effects (font (size 1.27 1.27)) hide)
-    )
-    (property "Value" "GND" (id 1) (at 122.174 57.3532 90))
-    (property "Footprint" "" (id 2) (at 122.047 52.959 0)
-      (effects (font (size 1.27 1.27)) hide)
-    )
-    (property "Datasheet" "" (id 3) (at 122.047 52.959 0)
-      (effects (font (size 1.27 1.27)) hide)
-    )
-    (pin "1")
-  )
   (symbol (lib_id "power:GND") (at 23.622 41.275 270) (unit 1)
     (in_bom yes) (on_board yes)
@@
     (pin "1")
   )
-  (symbol (lib_id "power:+3.3V") (at 114.427 46.609 90) (unit 1)
-    (in_bom yes) (on_board yes)
-    (property "Reference" "#PWR0316" (id 0) (at 118.237 46.609 0)
-      (effects (font (size 1.27 1.27)) hide)
-    )
-    (property "Value" "+3.3V" (id 1) (at 108.839 46.609 90))
-    (property "Footprint" "" (id 2) (at 114.427 46.609 0)
-      (effects (font (size 1.27 1.27)) hide)
-    )
-    (property "Datasheet" "" (id 3) (at 114.427 46.609 0)
-      (effects (font (size 1.27 1.27)) hide)
-    )
-    (pin "1")
+  (symbol (lib_id "Device:R") (at 160.02 30.48 0) (unit 1)
+    (in_bom yes) (on_board yes)
+    (property "Reference" "R?" (id 0) (at 156.21 29.21 0)
+      (effects (font (size 1.27 1.27)) (justify left))
+    )
+    (property "Value" "4.7k" (id 1) (at 154.94 31.75 0)
+      (effects (font (size 1.27 1.27)) (justify left))
+    )
+    (property "Footprint" "Resistor_SMD:R_0603_1608Metric" (id 2) (at 158.242 30.48 90)
+      (effects (font (size 1.27 1.27)) hide)
+    )
+    (property "Datasheet" "~" (id 3) (at 160.02 30.48 0)
+      (effects (font (size 1.27 1.27)) hide)
+    )
+    (pin "1")
+    (pin "2")
   )
   (symbol (lib_id "power:GND") (at 23.622 38.735 270) (unit 1)
@@
     (pin "1")
   )
+  (symbol (lib_id "Symbols:24AA02E48") (at 123.698 47.117 0) (unit 1)
+    (in_bom yes) (on_board yes) (fields_autoplaced)
+    (property "Reference" "U?" (id 0) (at 123.698 36.9275 0))
+    (property "Value" "24AA02E48" (id 1) (at 123.698 39.7026 0))
+    (property "Footprint" "Package_TO_SOT_SMD:SOT-23-5" (id 2) (at 123.698 36.957 0)
+      (effects (font (size 1.27 1.27)) hide)
+    )
+    (property "Datasheet" "" (id 3) (at 123.698 36.957 0)
+      (effects (font (size 1.27 1.27)) hide)
+    )
+    (pin "1")
+    (pin "2")
+    (pin "3")
+    (pin "4")
+    (pin "5")
+  )
   (symbol (lib_id "power:GND") (at 33.782 46.355 0) (unit 1)
     (in_bom yes) (on_board yes)
@@
     (pin "1")
   )
-  (symbol (lib_id "power:GND") (at 114.427 38.989 270) (unit 1)
-    (in_bom yes) (on_board yes)
-    (property "Reference" "#PWR0314" (id 0) (at 108.077 38.989 0)
-      (effects (font (size 1.27 1.27)) hide)
-    )
-    (property "Value" "GND" (id 1) (at 110.0328 39.116 90))
-    (property "Footprint" "" (id 2) (at 114.427 38.989 0)
-      (effects (font (size 1.27 1.27)) hide)
-    )
-    (property "Datasheet" "" (id 3) (at 114.427 38.989 0)
-      (effects (font (size 1.27 1.27)) hide)
-    )
-    (pin "1")
+  (symbol (lib_id "power:+3.3V") (at 160.02 26.67 0) (unit 1)
+    (in_bom yes) (on_board yes)
+    (property "Reference" "#PWR?" (id 0) (at 160.02 30.48 0)
+      (effects (font (size 1.27 1.27)) hide)
+    )
+    (property "Value" "+3.3V" (id 1) (at 160.02 22.86 0))
+    (property "Footprint" "" (id 2) (at 160.02 26.67 0)
+      (effects (font (size 1.27 1.27)) hide)
+    )
+    (property "Datasheet" "" (id 3) (at 160.02 26.67 0)
+      (effects (font (size 1.27 1.27)) hide)
+    )
+    (pin "1")
+  )
+  (symbol (lib_id "Device:R") (at 152.4 30.48 0) (unit 1)
+    (in_bom yes) (on_board yes)
+    (property "Reference" "R?" (id 0) (at 147.32 28.956 0)
+      (effects (font (size 1.27 1.27)) (justify left))
+    )
+    (property "Value" "4.7k" (id 1) (at 152.4 32.385 90)
+      (effects (font (size 1.27 1.27)) (justify left))
+    )
+    (property "Footprint" "Resistor_SMD:R_0603_1608Metric" (id 2) (at 150.622 30.48 90)
+      (effects (font (size 1.27 1.27)) hide)
+    )
+    (property "Datasheet" "~" (id 3) (at 152.4 30.48 0)
+      (effects (font (size 1.27 1.27)) hide)
+    )
+    (pin "1")
+    (pin "2")
   )
   (symbol (lib_id "power:GND") (at 118.491 25.527 270) (unit 1)
@@
       (effects (font (size 1.27 1.27)) hide)
     )
+    (pin "1")
+  )
+  (symbol (lib_id "power:+3.3V") (at 152.4 26.67 0) (unit 1)
+    (in_bom yes) (on_board yes)
+    (property "Reference" "#PWR?" (id 0) (at 152.4 30.48 0)
+      (effects (font (size 1.27 1.27)) hide)
+    )
+    (property "Value" "+3.3V" (id 1) (at 152.4 22.86 0))
+    (property "Footprint" "" (id 2) (at 152.4 26.67 0)
+      (effects (font (size 1.27 1.27)) hide)
+    )
+    (property "Datasheet" "" (id 3) (at 152.4 26.67 0)
+      (effects (font (size 1.27 1.27)) hide)
+    )
