File: GateWay_ver_2_2/PCB/Gateway_STM32_ver_2_2/COM PORT & BLE.kicad_sch (KiCad schematic)
At the start: 30 parts, among them J8 USB_B_Mini, U12 FT232RL, U14 SN74LV4052APW, U18 HC-05, U20 TPD2EUSB30

Commit message: 1
Parts:
- renumbered C88 to C102, C87 to C103, C86 to C104, C89 to C105, C90 to C106, C81 to C107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
