File: GateWay_ver_2_2/PCB/Gateway_STM32_ver_2_2/Ethernet.kicad_sch (KiCad schematic)
At the start: 42 parts, among them J2 HR911105A, U16 TPD2EUSB30, U4 W5500, U5 TPD2EUSB30, Y3 25mhz

Commit message: 1
Parts:
- renumbered C40 to C55, C42 to C56, C43 to C57, C44 to C58, C47 to C59, C48 to C60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
