File: GateWay_ver_2_2/PCB/Gateway_STM32_ver_2_2/Gateway_STM32_ver_2_0.kicad_sch (KiCad schematic)
At the start: 44 parts, among them J4 Conn_01x04, SW2 SW_Push, U7 STM32F407VETx, Y1 8mhz, Y2 Crystal_GND23

Commit message: 1
Parts:
- renumbered C46 to C1, C4 to C10, C5 to C11, C6 to C12, C7 to C13, C8 to C14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
Connections:
- net Nextion_Rx renamed DWIN_Rx
- net Nextion_Tx renamed DWIN_Tx
Other:
- added sheet Display (Display.kicad_sch)
