File: GateWay_ver_2_2/PCB/Gateway_STM32_ver_2_2/LTE.kicad_sch (KiCad schematic)
At the start: 44 parts, among them J3 SIM_Card, Q2 MMBT3904, Q3 AO3400, Q4 AO3400, Q9 AO3400, U6 SIM7600E-H

Commit message: 1
Parts:
- AE1, AE2: footprint Connector_Coaxial:SMA_Amphenol_901-144_Vertical -> Connector_Coaxial:SMA_Samtec_SMA-J-P-X-ST-EM1_EdgeMount
Changed lines of the file:
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@@
       (effects (font (size 1.27 1.27)) (justify left))
     )
-    (property "Footprint" "Connector_Coaxial:SMA_Amphenol_901-144_Vertical" (id 2) (at 241.808 107.823 0)
+    (property "Footprint" "Connector_Coaxial:SMA_Samtec_SMA-J-P-X-ST-EM1_EdgeMount" (id 2) (at 241.808 107.823 0)
       (effects (font (size 1.27 1.27)) hide)
     )
@@
       (effects (font (size 1.27 1.27)) (justify left))
     )
-    (property "Footprint" "Connector_Coaxial:SMA_Amphenol_901-144_Vertical" (id 2) (at 250.063 116.713 0)
-      (effects (font (size 1.27 1.27)) hide)
-    )
+    (property "Footprint" "Connector_Coaxial:SMA_Samtec_SMA-J-P-X-ST-EM1_EdgeMount" (id 2) (at 250.063 116.713 0)
+      (effects (font (size 1.27 1.27)) hide)
+    )

Commit message: 1
Parts:
- D21: renamed from D18; footprint Package_TO_SOT_SMD:SOT-363_SC-70-6_Handsoldering -> Package_TO_SOT_SMD:SOT-363_SC-70-6
- renumbered C60 to C73, C61 to C74, C62 to C75, C111 to C76, C112 to C77, C113 to C78, C63 to C79, C64 to C80, C65 to C81, C66 to C82, C67 to C83, C68 to C84, C69 to C85, D6 to D17, D7 to D18, D8 to D19, D9 to D20, J3 to J4, L4 to L6, Q9 to Q5, R32 to R43, R33 to R44, R42 to R45, R43 to R46, R44 to R47, R45 to R48, R46 to R49, R47 to R50, R48 to R51, R49 to R52, R96 to R53, R97 to R54, R50 to R55, R98 to R56, R51 to R57, R52 to R58, R53 to R59, U6 to U9
