File: GateWay_ver_2_2/PCB/Gateway_STM32_ver_2_2/Power.kicad_sch (KiCad schematic)
At the start: 66 parts, among them J1 DC-Jack_2.5x5.5, Q1 DMP3013SFV, U1 TPS54331, U19 RT8259, U2 RT8259, U3 RT8259

Commit message: 1
Parts:
- D13: renamed from D25; value SMAJ18.0CA -> SMAJ13.0CA
- renumbered C18 to C19, C19 to C20, C20 to C21, C21 to C22, C22 to C23, C13 to C24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
