File: GateWay_ver_2_2/PCB/Gateway_STM32_ver_2_2/RS-485 & 232.kicad_sch (KiCad schematic)
At the start: 37 parts, among them J12 RJ45_LED_Shielded, J6 RJ45_LED_Shielded, J7 RJ45_LED_Shielded, Q5 MMBT3906, Q6 MMBT3906, Q7 MMBT3906, Q8 MMBT3906, SW3 SW_Push, U10 MAX3485, U11 SN74LV4052APW, U9 MAX3232

Commit message: 1
Parts:
- added R114, R115: 510R, Resistor_SMD:R_0603_1608Metric, symbol Device:R
- R73: renamed from R61; value 220R -> 100R
- R75: renamed from R65; value 220R -> 100R
- renumbered C80 to C100, C76 to C101, C73 to C94, C74 to C95, C75 to C96, C77 to C97, C78 to C98, C79 to C99, D23 to D22, J6 to J8, J12 to J9, Q6 to Q10, Q5 to Q11, Q7 to Q8, Q8 to Q9, R58 to R70, R59 to R71, R60 to R72, R64 to R74, R73 to R76, R74 to R77, R63 to R78, R75 to R79, R82 to R80, R80 to R82, R62 to R84, R84 to R85, R78 to R86, U9 to U12, U10 to U13, U11 to U14
Connections:
- net +3V3: now also R115.2
- net 485_N: now also R114.2
- net 485_P: now also R115.1
- net GND: now also R114.1
