File: GateWay_ver_2_2/PCB/Gateway_STM32_ver_2_2/USB.kicad_sch (KiCad schematic)
At the start: 11 parts, among them J13 USB_A, U17 TPD2EUSB30, U21 TPS2041C

Commit message: 1
Parts:
- renumbered C107 to C117, C108 to C118, C109 to C119, C110 to C120, R92 to R110, R93 to R111, R94 to R112, R95 to R113, U21 to U26, U17 to U27
Changed lines of the file:
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@@
   (symbol (lib_id "power:+5V") (at 178.435 32.639 0) (unit 1)
     (in_bom yes) (on_board yes)
-    (property "Reference" "#PWR0169" (id 0) (at 178.435 36.449 0)
+    (property "Reference" "#PWR0364" (id 0) (at 178.435 36.449 0)
       (effects (font (size 1.27 1.27)) hide)
     )
@@
   (symbol (lib_id "power:GND") (at 140.208 72.39 0) (unit 1)
     (in_bom yes) (on_board yes)
-    (property "Reference" "#PWR0288" (id 0) (at 140.208 78.74 0)
+    (property "Reference" "#PWR0371" (id 0) (at 140.208 78.74 0)
       (effects (font (size 1.27 1.27)) hide)
     )
@@
   (symbol (lib_id "power:GND") (at 156.972 67.945 0) (unit 1)
     (in_bom yes) (on_board yes)
-    (property "Reference" "#PWR0174" (id 0) (at 156.972 74.295 0)
+    (property "Reference" "#PWR0369" (id 0) (at 156.972 74.295 0)
       (effects (font (size 1.27 1.27)) hide)
     )
@@
   (symbol (lib_id "power:+5V") (at 127.508 54.61 90) (unit 1)
     (in_bom yes) (on_board yes)
-    (property "Reference" "#PWR0173" (id 0) (at 131.318 54.61 0)
+    (property "Reference" "#PWR0368" (id 0) (at 131.318 54.61 0)
       (effects (font (size 1.27 1.27)) hide)
     )
@@
   (symbol (lib_id "power:GND") (at 206.502 91.44 0) (unit 1)
     (in_bom yes) (on_board yes)
-    (property "Reference" "#PWR037" (id 0) (at 206.502 97.79 0)
+    (property "Reference" "#PWR0373" (id 0) (at 206.502 97.79 0)
       (effects (font (size 1.27 1.27)) hide)
     )
@@
   (symbol (lib_id "power:+5V") (at 172.974 32.639 0) (unit 1)
     (in_bom yes) (on_board yes)
-    (property "Reference" "#PWR0167" (id 0) (at 172.974 36.449 0)
+    (property "Reference" "#PWR0363" (id 0) (at 172.974 36.449 0)
       (effects (font (size 1.27 1.27)) hide)
     )
@@
   (symbol (lib_id "power:GND") (at 172.974 40.259 0) (unit 1)
     (in_bom yes) (on_board yes)
-    (property "Reference" "#PWR0170" (id 0) (at 172.974 46.609 0)
+    (property "Reference" "#PWR0365" (id 0) (at 172.974 46.609 0)
       (effects (font (size 1.27 1.27)) hide)
     )
@@
   (symbol (lib_id "Device:C") (at 172.974 36.449 180) (unit 1)
     (in_bom yes) (on_board yes)
-    (property "Reference" "C107" (id 0) (at 169.799 32.639 90)
+    (property "Reference" "C117" (id 0) (at 169.799 32.639 90)
       (effects (font (size 1.27 1.27)) (justify left))
     )
@@
   (symbol (lib_id "Device:R") (at 189.738 80.137 90) (unit 1)
     (in_bom yes) (on_board yes)
-    (property "Reference" "R94" (id 0) (at 191.135 78.232 90)
+    (property "Reference" "R112" (id 0) (at 191.135 78.232 90)
       (effects (font (size 1.27 1.27)) (justify left))
     )
@@
   (symbol (lib_id "power:+5V") (at 113.411 49.53 0) (unit 1)
     (in_bom yes) (on_board yes)
-    (property "Reference" "#PWR0172" (id 0) (at 113.411 53.34 0)
+    (property "Reference" "#PWR0367" (id 0) (at 113.411 53.34 0)
       (effects (font (size 1.27 1.27)) hide)
     )
@@
   (symbol (lib_id "Device:C") (at 156.972 64.135 180) (unit 1)
     (in_bom yes) (on_board yes)
-    (property "Reference" "C109" (id 0) (at 153.797 60.325 90)
+    (property "Reference" "C119" (id 0) (at 153.797 60.325 90)
       (effects (font (size 1.27 1.27)) (justify left))
     )
@@
   (symbol (lib_id "Device:C") (at 162.433 64.135 0) (unit 1)
     (in_bom yes) (on_board yes)
-    (property "Reference" "C110" (id 0) (at 165.354 62.9666 90)
+    (property "Reference" "C120" (id 0) (at 165.354 62.9666 90)
       (effects (font (size 1.27 1.27)) (justify left))
     )
@@
   (symbol (lib_id "Device:R") (at 113.411 53.34 0) (unit 1)
     (in_bom yes) (on_board yes)
-    (property "Reference" "R92" (id 0) (at 115.189 52.1716 0)
+    (property "Reference" "R110" (id 0) (at 115.189 52.1716 0)
       (effects (font (size 1.27 1.27)) (justify left))
     )
@@
   (symbol (lib_id "power:GND") (at 182.753 126.238 0) (unit 1)
     (in_bom yes) (on_board yes)
-    (property "Reference" "#PWR0156" (id 0) (at 182.753 132.588 0)
+    (property "Reference" "#PWR0375" (id 0) (at 182.753 132.588 0)
       (effects (font (size 1.27 1.27)) hide)
     )
@@
   (symbol (lib_id "power:GND") (at 162.433 67.945 0) (unit 1)
     (in_bom yes) (on_board yes)
-    (property "Reference" "#PWR0238" (id 0) (at 162.433 74.295 0)
+    (property "Reference" "#PWR0370" (id 0) (at 162.433 74.295 0)
       (effects (font (size 1.27 1.27)) hide)
     )
@@
   (symbol (lib_id "Device:C") (at 178.435 36.449 0) (unit 1)
     (in_bom yes) (on_board yes)
-    (property "Reference" "C108" (id 0) (at 181.356 35.2806 90)
+    (property "Reference" "C118" (id 0) (at 181.356 35.2806 90)
       (effects (font (size 1.27 1.27)) (justify left))
     )
@@
   (symbol (lib_id "Symbols:TPS2041C") (at 140.208 58.42 0) (unit 1)
     (in_bom yes) (on_board yes) (fields_autoplaced)
-    (property "Reference" "U21" (id 0) (at 140.208 45.5635 0))
+    (property "Reference" "U26" (id 0) (at 140.208 45.5635 0))
     (property "Value" "TPS2041C" (id 1) (at 140.208 48.3386 0))
     (property "Footprint" "Package_TO_SOT_SMD:SOT-23-5" (id 2) (at 140.208 45.72 0)
@@
   (symbol (lib_id "Device:R") (at 189.738 84.074 90) (unit 1)
     (in_bom yes) (on_board yes)
-    (property "Reference" "R95" (id 0) (at 191.135 82.169 90)
+    (property "Reference" "R113" (id 0) (at 191.135 82.169 90)
       (effects (font (size 1.27 1.27)) (justify left))
     )
@@
   (symbol (lib_id "power:GND") (at 178.435 40.259 0) (unit 1)
     (in_bom yes) (on_board yes)
-    (property "Reference" "#PWR0171" (id 0) (at 178.435 46.609 0)
+    (property "Reference" "#PWR0366" (id 0) (at 178.435 46.609 0)
       (effects (font (size 1.27 1.27)) hide)
     )
@@
   (symbol (lib_id "power:GND") (at 209.042 91.44 0) (unit 1)
     (in_bom yes) (on_board yes)
-    (property "Reference" "#PWR038" (id 0) (at 209.042 97.79 0)
+    (property "Reference" "#PWR0374" (id 0) (at 209.042 97.79 0)
       (effects (font (size 1.27 1.27)) hide)
     )
@@
   (symbol (lib_id "Power_Protection:TPD2EUSB30") (at 182.753 116.078 0) (unit 1)
     (in_bom yes) (on_board yes) (fields_autoplaced)
-    (property "Reference" "U17" (id 0) (at 182.753 107.0315 0))
+    (property "Reference" "U27" (id 0) (at 182.753 107.0315 0))
     (property "Value" "TPD2EUSB30" (id 1) (at 182.753 109.8066 0))
     (property "Footprint" "Package_TO_SOT_SMD:Texas_DRT-3" (id 2) (at 163.703 123.698 0)
@@
   (symbol (lib_id "power:GND") (at 125.984 74.803 0) (unit 1)
     (in_bom yes) (on_board yes)
-    (property "Reference" "#PWR0289" (id 0) (at 125.984 81.153 0)
+    (property "Reference" "#PWR0372" (id 0) (at 125.984 81.153 0)
       (effects (font (size 1.27 1.27)) hide)
     )
@@
   (symbol (lib_id "Device:R") (at 125.984 70.993 0) (unit 1)
     (in_bom yes) (on_board yes)
-    (property "Reference" "R93" (id 0) (at 127.762 69.8246 0)
-      (effects (font (size 1.27 1.27)) (justify left))
-    )
+    (property "Reference" "R111" (id 0) (at 127.762 69.8246 0)
+      (effects (font (size 1.27 1.27)) (justify left))
+    )
