File: GateWay_ver_2_2/PCB/Gateway_STM32_ver_2_2/WIFI.kicad_sch (KiCad schematic)
At the start: 10 parts, among them J5 Conn_01x04, SW1 SW_Push, U8 ESP32-WROOM-32D

Commit message: 1
Parts:
- renumbered C70 to C86, C71 to C87, C72 to C88, R54 to R60, R55 to R61, R56 to R62, R57 to R63, SW1 to SW2, U8 to U10
Changed lines of the file:
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@@
   (symbol (lib_id "power:GND") (at 141.986 135.636 0) (unit 1)
     (in_bom yes) (on_board yes)
-    (property "Reference" "#PWR0284" (id 0) (at 141.986 141.986 0)
+    (property "Reference" "#PWR0219" (id 0) (at 141.986 141.986 0)
       (effects (font (size 1.27 1.27)) hide)
     )
@@
   (symbol (lib_id "power:GND") (at 177.546 65.151 90) (unit 1)
     (in_bom yes) (on_board yes)
-    (property "Reference" "#PWR0283" (id 0) (at 183.896 65.151 0)
+    (property "Reference" "#PWR0208" (id 0) (at 183.896 65.151 0)
       (effects (font (size 1.27 1.27)) hide)
     )
@@
   (symbol (lib_id "Device:C") (at 106.426 106.426 180) (unit 1)
     (in_bom yes) (on_board yes)
-    (property "Reference" "C72" (id 0) (at 111.506 108.966 0)
+    (property "Reference" "C88" (id 0) (at 111.506 108.966 0)
       (effects (font (size 1.27 1.27)) (justify left))
     )
@@
   (symbol (lib_id "Device:R") (at 118.491 64.516 180) (unit 1)
     (in_bom yes) (on_board yes)
-    (property "Reference" "R54" (id 0) (at 120.269 63.3476 0)
+    (property "Reference" "R60" (id 0) (at 120.269 63.3476 0)
       (effects (font (size 1.27 1.27)) (justify right))
     )
@@
   (symbol (lib_id "Device:R") (at 203.454 89.154 0) (unit 1)
     (in_bom yes) (on_board yes)
-    (property "Reference" "R56" (id 0) (at 205.232 87.9856 0)
+    (property "Reference" "R62" (id 0) (at 205.232 87.9856 0)
       (effects (font (size 1.27 1.27)) (justify left))
     )
@@
   (symbol (lib_id "Switch:SW_Push") (at 172.466 65.151 0) (unit 1)
     (in_bom yes) (on_board yes)
-    (property "Reference" "SW1" (id 0) (at 172.466 57.912 0))
+    (property "Reference" "SW2" (id 0) (at 172.466 57.912 0))
     (property "Value" "SW_Push" (id 1) (at 172.466 60.2234 0))
     (property "Footprint" "Button_Switch_SMD:SW_SPST_CK_RS282G05A3" (id 2) (at 172.466 60.071 0)
@@
   (symbol (lib_id "power:GND") (at 106.426 110.236 0) (unit 1)
     (in_bom yes) (on_board yes)
-    (property "Reference" "#PWR0285" (id 0) (at 106.426 116.586 0)
+    (property "Reference" "#PWR0216" (id 0) (at 106.426 116.586 0)
       (effects (font (size 1.27 1.27)) hide)
     )
@@
   (symbol (lib_id "Device:C") (at 98.171 106.426 0) (unit 1)
     (in_bom yes) (on_board yes)
-    (property "Reference" "C71" (id 0) (at 98.806 103.886 0)
+    (property "Reference" "C87" (id 0) (at 98.806 103.886 0)
       (effects (font (size 1.27 1.27)) (justify left))
     )
@@
   (symbol (lib_id "power:+3.3V") (at 118.491 60.706 0) (unit 1)
     (in_bom yes) (on_board yes)
-    (property "Reference" "#PWR0275" (id 0) (at 118.491 64.516 0)
+    (property "Reference" "#PWR0206" (id 0) (at 118.491 64.516 0)
       (effects (font (size 1.27 1.27)) hide)
     )
@@
   (symbol (lib_id "power:GND") (at 183.261 74.676 90) (unit 1)
     (in_bom yes) (on_board yes)
-    (property "Reference" "#PWR0281" (id 0) (at 189.611 74.676 0)
+    (property "Reference" "#PWR0209" (id 0) (at 189.611 74.676 0)
       (effects (font (size 1.27 1.27)) hide)
     )
@@
   (symbol (lib_id "power:+3.3V") (at 106.426 102.616 0) (unit 1)
     (in_bom yes) (on_board yes)
-    (property "Reference" "#PWR0279" (id 0) (at 106.426 106.426 0)
+    (property "Reference" "#PWR0214" (id 0) (at 106.426 106.426 0)
       (effects (font (size 1.27 1.27)) hide)
     )
@@
   (symbol (lib_id "power:+3.3V") (at 203.454 85.344 0) (unit 1)
     (in_bom yes) (on_board yes)
-    (property "Reference" "#PWR0280" (id 0) (at 203.454 89.154 0)
+    (property "Reference" "#PWR0211" (id 0) (at 203.454 89.154 0)
       (effects (font (size 1.27 1.27)) hide)
     )
@@
   (symbol (lib_id "power:+3.3V") (at 141.986 64.516 0) (unit 1)
     (in_bom yes) (on_board yes)
-    (property "Reference" "#PWR0274" (id 0) (at 141.986 68.326 0)
+    (property "Reference" "#PWR0207" (id 0) (at 141.986 68.326 0)
       (effects (font (size 1.27 1.27)) hide)
     )
@@
   (symbol (lib_id "power:GND") (at 118.491 79.756 0) (unit 1)
     (in_bom yes) (on_board yes)
-    (property "Reference" "#PWR0277" (id 0) (at 118.491 86.106 0)
+    (property "Reference" "#PWR0210" (id 0) (at 118.491 86.106 0)
       (effects (font (size 1.27 1.27)) hide)
     )
@@
   (symbol (lib_id "power:+3.3V") (at 98.171 102.616 0) (unit 1)
     (in_bom yes) (on_board yes)
-    (property "Reference" "#PWR0278" (id 0) (at 98.171 106.426 0)
+    (property "Reference" "#PWR0213" (id 0) (at 98.171 106.426 0)
       (effects (font (size 1.27 1.27)) hide)
     )
@@
   (symbol (lib_id "Device:R") (at 211.074 89.154 0) (unit 1)
     (in_bom yes) (on_board yes)
-    (property "Reference" "R57" (id 0) (at 212.852 87.9856 0)
+    (property "Reference" "R63" (id 0) (at 212.852 87.9856 0)
       (effects (font (size 1.27 1.27)) (justify left))
     )
@@
   (symbol (lib_id "power:GND") (at 200.406 118.491 270) (unit 1)
     (in_bom yes) (on_board yes)
-    (property "Reference" "#PWR0287" (id 0) (at 194.056 118.491 0)
+    (property "Reference" "#PWR0218" (id 0) (at 194.056 118.491 0)
       (effects (font (size 1.27 1.27)) hide)
     )
@@
   (symbol (lib_id "power:+3.3V") (at 211.074 85.344 0) (unit 1)
     (in_bom yes) (on_board yes)
-    (property "Reference" "#PWR0282" (id 0) (at 211.074 89.154 0)
+    (property "Reference" "#PWR0212" (id 0) (at 211.074 89.154 0)
       (effects (font (size 1.27 1.27)) hide)
     )
@@
   (symbol (lib_id "RF_Module:ESP32-WROOM-32D") (at 141.986 100.076 0) (unit 1)
     (in_bom yes) (on_board yes)
-    (property "Reference" "U8" (id 0) (at 154.051 63.881 0))
+    (property "Reference" "U10" (id 0) (at 154.051 63.881 0))
     (property "Value" "ESP32-WROOM-32D" (id 1) (at 154.051 65.786 0))
     (property "Footprint" "Footprint:ESP32-WROOM-32D" (id 2) (at 141.986 138.176 0)
@@
   (symbol (lib_id "Device:C") (at 118.491 75.946 180) (unit 1)
     (in_bom yes) (on_board yes)
-    (property "Reference" "C70" (id 0) (at 123.571 78.486 0)
+    (property "Reference" "C86" (id 0) (at 123.571 78.486 0)
       (effects (font (size 1.27 1.27)) (justify left))
     )
@@
   (symbol (lib_id "power:GND") (at 98.171 110.236 0) (unit 1)
     (in_bom yes) (on_board yes)
-    (property "Reference" "#PWR0276" (id 0) (at 98.171 116.586 0)
+    (property "Reference" "#PWR0215" (id 0) (at 98.171 116.586 0)
       (effects (font (size 1.27 1.27)) hide)
     )
@@
   (symbol (lib_id "power:+3.3V") (at 200.406 115.951 90) (unit 1)
     (in_bom yes) (on_board yes)
-    (property "Reference" "#PWR0286" (id 0) (at 204.216 115.951 0)
+    (property "Reference" "#PWR0217" (id 0) (at 204.216 115.951 0)
       (effects (font (size 1.27 1.27)) hide)
     )
@@
   (symbol (lib_id "Device:R") (at 179.451 74.676 90) (unit 1)
     (in_bom yes) (on_board yes)
-    (property "Reference" "R55" (id 0) (at 180.6194 76.454 0)
+    (property "Reference" "R61" (id 0) (at 180.6194 76.454 0)
       (effects (font (size 1.27 1.27)) (justify right))
     )
